File: 7Tally.kicad_pcb (KiCad board)
At the start: 2 copper layers, 54 x 37 mm, 50 parts, among them J2 B2B-PH-K-S_LF__SN_, P1 53047-0310, SW1 TL3300CF160Q, U1 ESP32-C3_SUPERMINI_TH, U2 BQ21040DBVR, U3 TC1263-3.3VOA

Commit message: fix(PCB): Small problem fixing
Parts:
- moved D10 0.25 mm to (83.2, 47.0)
- moved D11 0.25 mm to (88.2, 47.0)
- moved D12 0.25 mm to (53.2, 80.0)
- moved D13 0.25 mm to (58.2, 80.0)
- moved D14 0.25 mm to (63.2, 80.0)
- moved D15 0.25 mm to (68.2, 80.0)
- moved D16 0.25 mm to (73.2, 80.0)
- moved D17 0.25 mm to (78.2, 80.0)
- moved D18 0.25 mm to (83.2, 80.0)
- moved D19 0.25 mm to (88.2, 80.0)
- moved D3 0.25 mm to (78.2, 47.0)
- moved D5 0.25 mm to (73.2, 47.0)
- moved D6 0.25 mm to (63.2, 47.0)
- moved D7 0.25 mm to (68.2, 47.0)
- moved D8 0.25 mm to (58.2, 47.0)
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Routing:
- net Led_Vdd: track 51.2 -> 69.0 mm
- net NEOPIXEL_PIN: track 49.5 -> 44.2 mm, vias 3 -> 2
- net Net-(D19-DO): track 12.7 -> 8.85 mm
- net unconnected-(D9-DO-Pad1): track 0.00 -> 3.06 mm, vias 0 -> 3
- net Net-(D12-DI): track 11.8 -> 8.96 mm
- net Net-(D11-DI): track 11.9 -> 10.7 mm
- net VBAT: track 56.5 -> 55.9 mm
- net (no net): vias 2 -> 0
Other:
- outline, holes or cut-outs redrawn
- board text added: "*"
- board text added: "+"
- board text added: "."
- board text added: "BAT"
- board text added: "GP LED"
- board text added: "LDO"
- board text added: "NP"

Commit message: fix(PCB): pos-israel meet
Parts:
- moved C1 5.22 mm to (56.8, 65.5), turned to 90 degrees
- moved C3 1.39 mm to (56.8, 61.8)
Routing:
- net buttonPin: track 10.6 -> 13.8 mm
- net GND: track 2.56 -> 5.42 mm
- net Net-(D4-Pad2): track 42.8 -> 45.1 mm
- net VBAT: track 55.9 -> 57.8 mm
- net +3.3V: track 41.1 -> 39.8 mm
- net Net-(D2-K): track 16.1 -> 15.0 mm

Commit message: chore(PCB): Final Version
Parts:
- removed D4: ESD7351XV2T1G, ESD7351XV2T1G:SOD-523-2_ONSEMI
- added ?: , , F.Cu at (59.8, 50.5)
- added ?: , , F.Cu at (53.8, 76.5)
- added ?: , , F.Cu at (91.2, 56.0)
- added ?: , , F.Cu at (67.2, 76.5)
- added ?: , , F.Cu at (50.2, 69.5)
- added ?: , , F.Cu at (87.8, 50.5)
- added ?: , , F.Cu at (50.2, 57.5)
- added ?: , , F.Cu at (62.8, 50.5)
- added ?: , , F.Cu at (84.8, 50.5)
- added ?: , , F.Cu at (74.2, 50.5)
- added ?: , , F.Cu at (91.2, 68.0)
- added ?: , , F.Cu at (91.2, 57.5)
- added ?: , , F.Cu at (50.2, 71.0)
- added ?: , , F.Cu at (91.2, 69.5)
- added ?: , , F.Cu at (91.2, 52.5)
- added ?: , , F.Cu at (65.8, 50.5)
- added ?: , , F.Cu at (91.2, 65.0)
- added ?: , , F.Cu at (65.8, 76.5)
- added ?: , , F.Cu at (59.8, 76.5)
- added ?: , , F.Cu at (50.2, 66.5)
- added ?: , , F.Cu at (91.2, 60.5)
- added ?: , , F.Cu at (83.2, 50.5)
- added ?: , , F.Cu at (77.2, 50.5)
- added ?: , , F.Cu at (77.2, 76.5)
- added ?: , , F.Cu at (80.2, 50.5)
- added ?: , , F.Cu at (78.8, 76.5)
- added ?: , , F.Cu at (91.2, 66.5)
- added ?: , , F.Cu at (50.2, 52.5)
- added ?: , , F.Cu at (91.2, 59.0)
- added ?: , , F.Cu at (68.8, 76.5)
- added ?: , , F.Cu at (89.2, 76.5)
- added ?: , , F.Cu at (67.2, 50.5)
- added ?: , , F.Cu at (87.8, 76.5)
- added ?: , , F.Cu at (61.2, 50.5)
- added ?: , , F.Cu at (50.2, 74.5)
- added ?: , , F.Cu at (74.2, 76.5)
- added ?: , , F.Cu at (81.8, 76.5)
- added ?: , , F.Cu at (91.2, 74.5)
- added ?: , , F.Cu at (68.8, 50.5)
- added ?: , , F.Cu at (52.2, 76.5)
- added ?: , , F.Cu at (52.2, 50.5)
- added ?: , , F.Cu at (50.2, 59.0)
- added ?: , , F.Cu at (75.8, 76.5)
- added ?: , , F.Cu at (84.8, 76.5)
- added ?: , , F.Cu at (72.8, 76.5)
- added ?: , , F.Cu at (72.8, 50.5)
- added ?: , , F.Cu at (80.2, 76.5)
- added ?: , , F.Cu at (53.8, 50.5)
- added ?: , , F.Cu at (50.2, 68.0)
- added ?: , , F.Cu at (58.2, 50.5)
- added ?: , , F.Cu at (81.8, 50.5)
- added ?: , , F.Cu at (50.2, 56.0)
- added ?: , , F.Cu at (91.2, 71.0)
- added ?: , , F.Cu at (78.8, 50.5)
- added ?: , , F.Cu at (50.2, 60.5)
- added ?: , , F.Cu at (58.2, 76.5)
- added ?: , , F.Cu at (50.2, 62.0)
- added ?: , , F.Cu at (83.2, 76.5)
- added ?: , , F.Cu at (75.8, 50.5)
- added ?: , , F.Cu at (61.2, 76.5)
- added ?: , , F.Cu at (62.8, 76.5)
- added C-Edge-1mmx2mmx0.8mmTH: , Library:C-Edge-1mmx2mmx0.8mmTH, F.Cu at (91.2, 62.0)
- added C-Edge-1mmx2mmx0.8mmTH: , Library:C-Edge-1mmx2mmx0.8mmTH, F.Cu at (89.2, 50.5)
- added C-Edge-1mmx2mmx0.8mmTH: , Library:C-Edge-1mmx2mmx0.8mmTH, F.Cu at (64.2, 50.5)
- added C-Edge-1mmx2mmx0.8mmTH: , Library:C-Edge-1mmx2mmx0.8mmTH, F.Cu at (64.2, 76.5)
- added C-Edge-1mmx2mmx0.8mmTH: , Library:C-Edge-1mmx2mmx0.8mmTH, F.Cu at (56.8, 76.5)
- added C-Edge-1mmx2mmx0.8mmTH: , Library:C-Edge-1mmx2mmx0.8mmTH, F.Cu at (50.2, 65.0)
- added C-Edge-1mmx2mmx0.8mmTH: , Library:C-Edge-1mmx2mmx0.8mmTH, F.Cu at (56.8, 50.5)
- added C10: 0.4u, Capacitor_SMD:C_0201_0603Metric, F.Cu at (50.8, 79.5)
- added C11: 0.2u, Capacitor_SMD:C_0201_0603Metric, F.Cu at (46.0, 51.0)
- added C12: 0.2u, Capacitor_SMD:C_0201_0603Metric, F.Cu at (45.0, 76.0)
- added C5: 0.4u, Capacitor_SMD:C_0201_0603Metric, F.Cu at (90.8, 47.5)
- added C6: 0.4u, Capacitor_SMD:C_0201_0603Metric, F.Cu at (50.8, 46.5)
- added C7: 0.2u, Capacitor_SMD:C_0201_0603Metric, F.Cu at (96.0, 51.0)
- added C8: 0.2u, Capacitor_SMD:C_0201_0603Metric, F.Cu at (94.9, 76.0)
- added C9: 0.4u, Capacitor_SMD:C_0201_0603Metric, F.Cu at (90.8, 80.5)
- added D30: US1A, US1A:DIOM4325X250N, B.Cu at (59.8, 68.2)
- moved C2 2.58 mm to (53.5, 61.0)
- moved R9 1.64 mm to (53.5, 64.8)
- moved C1 0.80 mm to (56.8, 64.7)
- moved C3 0.80 mm to (56.8, 61.0)
- moved U3 0.50 mm to (61.0, 63.0)
- moved C4 0.17 mm to (61.0, 58.2)
Routing:
- net Led_Vdd: track 69.3 -> 83.2 mm, vias 50 -> 22
- net enablePort: track 26.7 -> 24.0 mm
- net +5V: track 21.8 -> 24.4 mm
- net Net-(D30-PadA): track 45.1 -> 42.7 mm
- net Net-(D11-DI): track 10.7 -> 8.50 mm, vias 5 -> 2
- net Net-(D12-DI): track 8.96 -> 7.10 mm, vias 5 -> 2
- net Net-(D19-DO): track 8.85 -> 7.04 mm, vias 5 -> 2
- net GND: track 5.42 -> 3.73 mm, vias 48 -> 20
- net NEOPIXEL_PIN: track 44.4 -> 43.0 mm, vias 2 -> 1
- net VBAT: track 57.8 -> 56.8 mm
- net Net-(D2-K): track 15.0 -> 15.6 mm
- net +3.3V: track 39.8 -> 39.2 mm
- net unconnected-(D9-DO-Pad1): track 3.06 -> 2.56 mm, vias 3 -> 1
Other:
- board text added: "7Tally"
- board text added: "Miguel Velo"
- board text added: "Zé Mateus"
