File: 7Tally.kicad_sch (KiCad schematic)
At the start: 24 parts, among them J2 B2B-PH-K-S_LF__SN_, P1 53047-0310, SW1 TL3300CF160Q, U1 ESP32-C3_SUPERMINI_TH, U2 BQ21040DBVR, U3 TC1263-3.3VOA

Commit message: fix(PCB): pos-israel meet
Other:
- moved on the sheet: C3, C4
Changed lines of the file:
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@@
 	(wire
 		(pts
-			(xy 261.62 50.8) (xy 261.62 45.72)
+			(xy 242.57 129.54) (xy 242.57 124.46)
 		)
 		(stroke
@@
 	(wire
 		(pts
-			(xy 261.62 58.42) (xy 261.62 63.5)
+			(xy 242.57 137.16) (xy 242.57 142.24)
 		)
 		(stroke
@@
 	(wire
 		(pts
-			(xy 248.92 50.8) (xy 248.92 45.72)
+			(xy 257.81 55.88) (xy 257.81 50.8)
 		)
 		(stroke
@@
 	(wire
 		(pts
-			(xy 248.92 58.42) (xy 248.92 63.5)
+			(xy 257.81 63.5) (xy 257.81 68.58)
 		)
 		(stroke
@@
 	(global_label "BP"
 		(shape input)
-		(at 261.62 45.72 90)
+		(at 242.57 124.46 90)
 		(fields_autoplaced yes)
 		(effects
@@
 		)
 		(property "Intersheetrefs" "${INTERSHEET_REFS}"
-			(at 261.62 40.1948 90)
+			(at 242.57 118.9348 90)
 			(effects
 				(font
@@
 	(symbol
 		(lib_id "Device:C")
-		(at 248.92 54.61 0)
+		(at 257.81 59.69 0)
 		(unit 1)
 		(exclude_from_sim no)
@@
 		(fields_autoplaced yes)
 		(property "Reference" "C3"
-			(at 252.73 53.3399 0)
+			(at 261.62 58.4199 0)
 			(effects
 				(font
@@
 		)
 		(property "Value" "1u"
-			(at 252.73 55.8799 0)
+			(at 261.62 60.9599 0)
 			(effects
 				(font
@@
 		)
 		(property "Footprint" "Capacitor_SMD:C_0805_2012Metric"
-			(at 249.8852 58.42 0)
+			(at 258.7752 63.5 0)
 			(effects
 				(font
@@
 		)
 		(property "Datasheet" "~"
-			(at 248.92 54.61 0)
+			(at 257.81 59.69 0)
 			(effects
 				(font
@@
 		)
 		(property "Description" "Unpolarized capacitor"
-			(at 248.92 54.61 0)
+			(at 257.81 59.69 0)
 			(effects
 				(font
@@
 	(symbol
 		(lib_id "Device:C")
-		(at 261.62 54.61 0)
+		(at 242.57 133.35 0)
 		(unit 1)
 		(exclude_from_sim no)
@@
 		(fields_autoplaced yes)
 		(property "Reference" "C4"
-			(at 265.43 53.3399 0)
+			(at 246.38 132.0799 0)
 			(effects
 				(font
@@
 		)
 		(property "Value" "470p"
-			(at 265.43 55.8799 0)
+			(at 246.38 134.6199 0)
 			(effects
 				(font
@@
 		)
 		(property "Footprint" "Capacitor_SMD:C_0805_2012Metric"
-			(at 262.5852 58.42 0)
+			(at 243.5352 137.16 0)
 			(effects
 				(font
@@
 		)
 		(property "Datasheet" "~"
-			(at 261.62 54.61 0)
+			(at 242.57 133.35 0)
 			(effects
 				(font
@@
 		)
 		(property "Description" "Unpolarized capacitor"
-			(at 261.62 54.61 0)
+			(at 242.57 133.35 0)
 			(effects
 				(font
@@
 	(symbol
 		(lib_id "power:+3.3V")
-		(at 248.92 45.72 0)
+		(at 257.81 50.8 0)
 		(unit 1)
 		(exclude_from_sim no)
@@
 		(fields_autoplaced yes)
 		(property "Reference" "#PWR020"
-			(at 248.92 49.53 0)
+			(at 257.81 54.61 0)
 			(effects
 				(font
@@
 		)
 		(property "Value" "+3.3V"
-			(at 248.92 40.64 0)
+			(at 257.81 45.72 0)
 			(effects
 				(font
@@
 		)
 		(property "Footprint" ""
-			(at 248.92 45.72 0)
+			(at 257.81 50.8 0)
 			(effects
 				(font
@@
 		)
 		(property "Datasheet" ""
-			(at 248.92 45.72 0)
+			(at 257.81 50.8 0)
 			(effects
 				(font
@@
 		)
 		(property "Description" "Power symbol creates a global label with name \"+3.3V\""
-			(at 248.92 45.72 0)
+			(at 257.81 50.8 0)
 			(effects
 				(font
@@
 	(symbol
 		(lib_id "power:GND")
-		(at 248.92 63.5 0)
+		(at 257.81 68.58 0)
 		(unit 1)
 		(exclude_from_sim no)
@@
 		(fields_autoplaced yes)
 		(property "Reference" "#PWR021"
-			(at 248.92 69.85 0)
+			(at 257.81 74.93 0)
 			(effects
 				(font
@@
 		)
 		(property "Value" "GND"
-			(at 248.92 68.58 0)
+			(at 257.81 73.66 0)
 			(effects
 				(font
@@
 		)
 		(property "Footprint" ""
-			(at 248.92 63.5 0)
+			(at 257.81 68.58 0)
 			(effects
 				(font
@@
 		)
 		(property "Datasheet" ""
-			(at 248.92 63.5 0)
+			(at 257.81 68.58 0)
 			(effects
 				(font
@@
 		)
 		(property "Description" "Power symbol creates a global label with name \"GND\" , ground"
-			(at 248.92 63.5 0)
+			(at 257.81 68.58 0)
 			(effects
 				(font
@@
 	(symbol
 		(lib_id "power:GND")
-		(at 261.62 63.5 0)
+		(at 242.57 142.24 0)
 		(unit 1)
 		(exclude_from_sim no)
@@
 		(fields_autoplaced yes)
 		(property "Reference" "#PWR023"
-			(at 261.62 69.85 0)
+			(at 242.57 148.59 0)
 			(effects
 				(font
@@
 		)
 		(property "Value" "GND"
-			(at 261.62 68.58 0)
+			(at 242.57 147.32 0)
 			(effects
 				(font
@@
 		)
 		(property "Footprint" ""
-			(at 261.62 63.5 0)
+			(at 242.57 142.24 0)
 			(effects
 				(font
@@
 		)
 		(property "Datasheet" ""
-			(at 261.62 63.5 0)
+			(at 242.57 142.24 0)
 			(effects
 				(font
@@
 		)
 		(property "Description" "Power symbol creates a global label with name \"GND\" , ground"
-			(at 261.62 63.5 0)
+			(at 242.57 142.24 0)
 			(effects
 				(font

Commit message: chore(PCB): Final Version
Parts:
- removed D4: ESD7351XV2T1G, ESD7351XV2T1G:SOD-523-2_ONSEMI, symbol ESD7351XV2T1G:ESD7351XV2T1G
- added D30: US1A, US1A:DIOM4325X250N, symbol US1A:US1A
Connections:
- net enablePort: now also D30.C
- net at R5.1, SW1.3, SW1.4: now also D30.A
